File: Halogen discharger/Halogen discharger.kicad_pcb (KiCad board)
At the start: 2 copper layers, 63.5 x 54.6 mm, 22 parts, among them J1 Conn_01x02, J2 Conn_01x02, J3 Conn_01x01, J4 Conn_01x01, J5 Conn_01x01, J6 Conn_01x01

Commit message: Halogen discharger updates.
Parts:
- removed J6: Conn_01x01, Library:SolderWirePad_1x01_SMD_2x4mm
- added REF**: Cable tie hole, Library:Cable tie hole, F.Cu at (165.1, 153.0)
- added REF**: Cable tie hole, Library:Cable tie hole, F.Cu at (149.9, 153.0)
- J2: value Conn_01x02 -> Conn_01x01; footprint Connector_AMASS:AMASS_XT30PW-F_1x02_P2.50mm_Horizontal -> Connector_Wire:SolderWirePad_1x01_SMD_1x2mm
- J3, J4, J5: footprint Library:SolderWirePad_1x01_SMD_2x4mm -> Connector_Wire:SolderWirePad_1x01_SMD_1x2mm
- moved J4 62.4 mm to (181.6, 104.1), turned to 180 degrees
- moved J2 62.0 mm to (133.3, 104.1), turned to 0 degrees
- moved J5 49.5 mm to (179.1, 104.1), turned to 180 degrees
- moved J3 48.9 mm to (135.9, 104.1)
- moved J1 17.1 mm to (160.0, 148.0)
Connections:
- J1 pad 1: Net-(J1-Pad1) -> GND
- J1 pad 2: Net-(J1-Pad2) -> VCC
- J2 pad 1: Net-(J2-Pad1) -> VCC
- J3 pad 1: Net-(J1-Pad2) -> GND
- J4 pad 1: Net-(J1-Pad1) -> VCC
- J5 pad 1: Net-(J1-Pad2) -> GND
- LA1 pad 2: Net-(J1-Pad2) -> VCC
- LA10 pad 1: Net-(J1-Pad1) -> Net-(LA10-Pad1)
- LA10 pad 2: Net-(LA10-Pad2) -> Net-(LA1-Pad1)
- LA11 pad 2: Net-(J1-Pad1) -> Net-(LA10-Pad1)
- LA12 pad 1: Net-(J2-Pad1) -> GND
- LA2 pad 1: Net-(J1-Pad1) -> Net-(LA10-Pad1)
- LA3 pad 1: Net-(LA3-Pad1) -> Net-(LA11-Pad1)
- LA3 pad 2: Net-(J1-Pad1) -> Net-(LA10-Pad1)
- LA4 pad 1: Net-(J2-Pad1) -> GND
- LA4 pad 2: Net-(LA3-Pad1) -> Net-(LA11-Pad1)
- LA5 pad 1: Net-(LA5-Pad1) -> Net-(LA1-Pad1)
- LA5 pad 2: Net-(J1-Pad2) -> VCC
- LA6 pad 1: Net-(J1-Pad1) -> Net-(LA10-Pad1)
- LA6 pad 2: Net-(LA5-Pad1) -> Net-(LA1-Pad1)
- LA7 pad 1: Net-(LA7-Pad1) -> Net-(LA11-Pad1)
- LA7 pad 2: Net-(J1-Pad1) -> Net-(LA10-Pad1)
- LA8 pad 1: Net-(J2-Pad1) -> GND
- LA8 pad 2: Net-(LA7-Pad1) -> Net-(LA11-Pad1)
- LA9 pad 1: Net-(LA10-Pad2) -> Net-(LA1-Pad1)
- LA9 pad 2: Net-(J1-Pad2) -> VCC
Routing:
- net Net-(LA10-Pad1): track 0.00 -> 188.6 mm
- net Net-(LA1-Pad1): track 5.08 -> 169.7 mm
- net Net-(LA11-Pad1): track 5.08 -> 169.7 mm
- net Net-(J1-Pad2): track 132.7 -> 0.00 mm
- net Net-(J1-Pad1): track 84.5 -> 0.00 mm
- net Net-(J2-Pad1): track 45.2 -> 0.00 mm
- net Net-(LA5-Pad1): track 5.08 -> 0.00 mm
- net Net-(LA10-Pad2): track 5.08 -> 0.00 mm
- net Net-(LA7-Pad1): track 5.08 -> 0.00 mm
- net Net-(LA3-Pad1): track 5.08 -> 0.00 mm
- net GND: track 0.00 -> 3.59 mm, vias 0 -> 2
- added copper zone on B.Cu, net GND
- added copper zone on B.Cu, net Net-(LA10-Pad1)
- added copper zone on F.Cu, net Net-(LA10-Pad1)
- added copper zone on F.Cu, net VCC
Other:
- board text added: "+"
- board text added: "-"
- board text removed: "CONNECT ONE ONLY"
- board text removed: "x12"
- board text removed: "x6"
